Commit message: Fixed bash script for launching a new robot. Rearraging things inside the WS in order to automate the robots launching. Right now the system is working well baxter and pr2.

File: django/static/atlas_description/atlas.urdf (robot description, URDF)
Before this commit: robot drc_skeleton, 28 links, 28 joints
Links:
- link l_clav: geometry collision mesh filename=package://atlas_description/meshes/l_clav.stl scale=1 1 1; visual mesh filename=package://atlas_description/meshes/l_clav.dae scale=1 1 1
- link l_farm: geometry collision mesh filename=package://atlas_description/meshes/l_farm.stl scale=1 1 1; visual mesh filename=package://atlas_description/meshes/l_farm.dae scale=1 1 1
- link l_foot: geometry collision mesh filename=package://atlas_description/meshes/l_foot.stl scale=1 1 1; visual mesh filename=package://atlas_description/meshes/l_foot.dae scale=1 1 1
- link l_hand: geometry collision mesh filename=package://atlas_description/meshes/l_hand.stl scale=1 1 1; visual mesh filename=package://atlas_description/meshes/l_hand.dae scale=1 1 1
- link l_larm: geometry collision mesh filename=package://atlas_description/meshes/l_larm.stl scale=1 1 1; visual mesh filename=package://atlas_description/meshes/l_larm.dae scale=1 1 1
- link l_lglut: geometry collision mesh filename=package://atlas_description/meshes/l_lglut.stl scale=1 1 1; visual mesh filename=package://atlas_description/meshes/l_lglut.dae scale=1 1 1
- link l_lleg: geometry collision mesh filename=package://atlas_description/meshes/l_lleg.stl scale=1 1 1; visual mesh filename=package://atlas_description/meshes/l_lleg.dae scale=1 1 1
- link l_scap: geometry collision mesh filename=package://atlas_description/meshes/l_scap.stl scale=1 1 1; visual mesh filename=package://atlas_description/meshes/l_scap.dae scale=1 1 1
- link l_talus: geometry collision mesh filename=package://atlas_description/meshes/l_talus.stl scale=1 1 1; visual mesh filename=package://atlas_description/meshes/l_talus.dae scale=1 1 1
- link l_uarm: geometry collision mesh filename=package://atlas_description/meshes/l_uarm.stl scale=1 1 1; visual mesh filename=package://atlas_description/meshes/l_uarm.dae scale=1 1 1
- link l_uglut: geometry collision mesh filename=package://atlas_description/meshes/l_uglut.stl scale=1 1 1; visual mesh filename=package://atlas_description/meshes/l_uglut.dae scale=1 1 1
- link l_uleg: geometry collision mesh filename=package://atlas_description/meshes/l_uleg.stl scale=1 1 1; visual mesh filename=package://atlas_description/meshes/l_uleg.dae scale=1 1 1
- link ltorso: geometry collision mesh filename=package://atlas_description/meshes/ltorso.stl scale=1 1 1; visual mesh filename=package://atlas_description/meshes/ltorso.dae scale=1 1 1
- link mtorso: geometry collision mesh filename=package://atlas_description/meshes/mtorso.stl scale=1 1 1; visual mesh filename=package://atlas_description/meshes/mtorso.dae scale=1 1 1
- link pelvis: geometry collision mesh filename=package://atlas_description/meshes/pelvis.stl scale=1 1 1; visual mesh filename=package://atlas_description/meshes/pelvis.dae scale=1 1 1
- link r_clav: geometry collision mesh filename=package://atlas_description/meshes/r_clav.stl scale=1 1 1; visual mesh filename=package://atlas_description/meshes/r_clav.dae scale=1 1 1
- link r_farm: geometry collision mesh filename=package://atlas_description/meshes/r_farm.stl scale=1 1 1; visual mesh filename=package://atlas_description/meshes/r_farm.dae scale=1 1 1
- link r_foot: geometry collision mesh filename=package://atlas_description/meshes/r_foot.stl scale=1 1 1; visual mesh filename=package://atlas_description/meshes/r_foot.dae scale=1 1 1
- link r_hand: geometry collision mesh filename=package://atlas_description/meshes/r_hand.stl scale=1 1 1; visual mesh filename=package://atlas_description/meshes/r_hand.dae scale=1 1 1
- link r_larm: geometry collision mesh filename=package://atlas_description/meshes/r_larm.stl scale=1 1 1; visual mesh filename=package://atlas_description/meshes/r_larm.dae scale=1 1 1
- link r_lglut: geometry collision mesh filename=package://atlas_description/meshes/r_lglut.stl scale=1 1 1; visual mesh filename=package://atlas_description/meshes/r_lglut.dae scale=1 1 1
- link r_lleg: geometry collision mesh filename=package://atlas_description/meshes/r_lleg.stl scale=1 1 1; visual mesh filename=package://atlas_description/meshes/r_lleg.dae scale=1 1 1
- link r_scap: geometry collision mesh filename=package://atlas_description/meshes/r_scap.stl scale=1 1 1; visual mesh filename=package://atlas_description/meshes/r_scap.dae scale=1 1 1
- link r_talus: geometry collision mesh filename=package://atlas_description/meshes/r_talus.stl scale=1 1 1; visual mesh filename=package://atlas_description/meshes/r_talus.dae scale=1 1 1
- link r_uarm: geometry collision mesh filename=package://atlas_description/meshes/r_uarm.stl scale=1 1 1; visual mesh filename=package://atlas_description/meshes/r_uarm.dae scale=1 1 1
- link r_uglut: geometry collision mesh filename=package://atlas_description/meshes/r_uglut.stl scale=1 1 1; visual mesh filename=package://atlas_description/meshes/r_uglut.dae scale=1 1 1
- link r_uleg: geometry collision mesh filename=package://atlas_description/meshes/r_uleg.stl scale=1 1 1; visual mesh filename=package://atlas_description/meshes/r_uleg.dae scale=1 1 1
- link utorso: geometry collision mesh filename=package://atlas_description/meshes/utorso.stl scale=1 1 1; visual mesh filename=package://atlas_description/meshes/utorso.dae scale=1 1 1

Commit message: Added fixed r2_description. Fixed atlas_description issues. tweaked bridge.py and move_group.launch

File: django/static/atlas_description/atlas.urdf (robot description, URDF)
Before this commit: robot drc_skeleton, 28 links, 28 joints
Joints:
- removed joint neck_ay
